Commit message: update

File: msp_sim/urdf/lidar.urdf.xacro (robot description, xacro)
@@ -3,6 +3,6 @@
   <link name="lidar" />
   <xacro:include filename="$(find msp_sim)/urdf/mid360.urdf.xacro" />
-  <xacro:Livox_Mid360 parent="mid360_mount_plate"  topic="/livox/lidar"  hz="5" samples="20000" gpu_enabled ="1">
-    <origin xyz="0 0 0.0063" rpy="0 0 0" />
+  <xacro:Livox_Mid360 parent="lidar" topic="/livox/lidar"  hz="5" samples="20000" gpu_enabled ="1">
+    <origin xyz="0 0 0.0063" rpy="0 0.35 0" />
   </xacro:Livox_Mid360>
 </robot>

Commit message: add sim test

File: msp_sim/urdf/lidar.urdf.xacro (robot description, xacro)
@@ -4,5 +4,5 @@
   <xacro:include filename="$(find msp_sim)/urdf/mid360.urdf.xacro" />
   <xacro:Livox_Mid360 parent="lidar" topic="/livox/lidar"  hz="5" samples="20000" gpu_enabled ="1">
-    <origin xyz="0 0 0.0063" rpy="0 0.35 0" />
+    <origin xyz="0 0 0.0063" rpy="0 0 0" />
   </xacro:Livox_Mid360>
 </robot>

File: msp_sim/urdf/mid360_mount.urdf.xacro (robot description, xacro)
@@ -78,5 +78,6 @@
   <xacro:Livox_Mid360 parent="mid360_mount_plate"  topic="${topic}"  hz="${hz}" samples="${samples}" gpu_enabled ="${gpu_enabled}">
     <!-- <origin xyz="-0.016 0 0" rpy="0 0.35 0" /> -->
-    <origin xyz="0 0 0" rpy="0 0 0" />
+    <!-- <origin xyz="0 0 0" rpy="0 0 0" /> -->
+    <xacro:insert_block name="origin" />
   </xacro:Livox_Mid360>
   </xacro:macro>
